File: h-bridge/_autosave-h-bridge.kicad_sch (KiCad schematic)
At the start: 29 parts, among them J1 Screw_Terminal_01x06, Q1 IRF4905, Q2 IRLZ44N, Q3 IRF4905, Q4 IRLZ44N, Q5 2N2222, Q6 2N2222, Q7 IRF4905, Q8 IRF4905

Commit message: gerber files done
Parts:
- renumbered C3 to C1, D9 to D1, D10 to D2, D15 to D3, D16 to D4, D1 to D5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
